Commit message: added extra lidar

File: urdf/catvehicle_lidars.xacro (robot description, xacro)
@@ -3,7 +3,7 @@
         <xacro:include filename="$(find catvehicle)/urdf/catvehicle_top_centre_lidar.gazebo"/>
         <!-- <xacro:include filename="$(find catvehicle)/urdf/catvehicle_top_left_lidar.gazebo"/>
-        <xacro:include filename="$(find catvehicle)/urdf/catvehicle_top_right_lidar.gazebo"/>
+        <xacro:include filename="$(find catvehicle)/urdf/catvehicle_top_right_lidar.gazebo"/> -->
         <xacro:include filename="$(find catvehicle)/urdf/catvehicle_rear_centre_lidar.gazebo"/>
-        <xacro:include filename="$(find catvehicle)/urdf/catvehicle_rear_left_lidar.gazebo"/>
+        <!-- <xacro:include filename="$(find catvehicle)/urdf/catvehicle_rear_left_lidar.gazebo"/>
         <xacro:include filename="$(find catvehicle)/urdf/catvehicle_rear_right_lidar.gazebo"/> -->
         <!-- TOP CENTRE LIDAR -->
@@ -92,6 +92,6 @@
         </link> -->
         <!-- REAR CENTRE LIDAR -->
-        <!-- <joint name="rear_centre_lidar_joint" type="fixed">
-            <origin xyz="${-10*camera_box} 0 ${car_height + 2*sensor_box + 0.01}" rpy="0 0 ${PI}"/>
+        <joint name="rear_centre_lidar_joint" type="fixed">
+            <origin xyz="${-12*camera_box} 0 ${car_height + 2*sensor_box + 0.01}" rpy="0 0 ${PI}"/>
             <axis xyz="0 0 1"/>
             <parent link="base_link"/>
@@ -118,5 +118,5 @@
                 izz="${(1/6)*front_laser_mass*front_laser_size*front_laser_size}" />
             </inertial>
-        </link> -->
+        </link>
         <!-- REAR LEFT LIDAR -->
         <!-- <joint name="rear_left_lidar_joint" type="fixed">
